File: neopixel_cab_lights/neopixel_cab_lights.brd (EAGLE design)
At the start: 100 x 80 mm, 10 parts

Commit message: Eagle BRD & SCH files update.. Still working on board
Parts:
- moved PAD1 51.6 mm to (20.8, 32.3)
- moved JP2 48.6 mm to (22.9, 22.4), turned to 270 degrees
- moved PAD3 47.0 mm to (22.9, 32.3)
- moved JP1 37.2 mm to (10.2, 22.4), turned to 270 degrees
- moved PAD2 36.6 mm to (18.8, 32.3)
- moved C1 32.1 mm to (5.08, 9.91), turned to 180 degrees
- moved R2 30.4 mm to (10.9, 31.8)
- moved R1 25.4 mm to (6.35, 20.1), turned to 270 degrees
- moved S1 22.4 mm to (4.57, 3.30), turned to 180 degrees
Routing:
- net 5V+REG: track 0.00 -> 4.97 mm
- net DIN: track 0.00 -> 3.00 mm
- added copper zone on layer 1, net GND
- added copper zone on layer 16, net N$1
Other:
- board size 100 x 80 mm -> 24.9 x 33.3 mm
Changed lines of the file:
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@@
 <?xml version="1.0" encoding="utf-8"?>
 <!DOCTYPE eagle SYSTEM "eagle.dtd">
-<eagle version="7.5.0">
+<eagle version="6.5.0">
 <drawing>
 <settings>
@@
 <setting verticaltext="up"/>
 </settings>
-<grid distance="0.05" unitdist="inch" unit="inch" style="lines" multiple="1" display="no" altdistance="0.025" altunitdist="inch" altunit="inch"/>
+<grid distance="0.01" unitdist="inch" unit="inch" style="lines" multiple="1" display="yes" altdistance="0.001" altunitdist="inch" altunit="inch"/>
 <layers>
 <layer number="1" name="Top" color="4" fill="1" visible="yes" active="yes"/>
@@
 <board>
 <plain>
-<wire x1="0" y1="0" x2="100" y2="0" width="0" layer="20"/>
-<wire x1="100" y1="0" x2="100" y2="80" width="0" layer="20"/>
-<wire x1="100" y1="80" x2="0" y2="80" width="0" layer="20"/>
-<wire x1="0" y1="80" x2="0" y2="0" width="0" layer="20"/>
+<wire x1="8.89" y1="1.524" x2="8.89" y2="27.686" width="0" layer="21"/>
+<wire x1="8.89" y1="27.686" x2="9.652" y2="28.448" width="0" layer="21"/>
+<wire x1="9.652" y1="28.448" x2="12.954" y2="28.448" width="0" layer="21"/>
+<wire x1="12.954" y1="28.448" x2="14.478" y2="29.972" width="0" layer="21"/>
+<wire x1="14.478" y1="29.972" x2="21.59" y2="29.972" width="0" layer="21"/>
+<wire x1="21.59" y1="29.972" x2="23.368" y2="28.194" width="0" layer="21"/>
+<wire x1="23.368" y1="28.194" x2="24.13" y2="28.194" width="0" layer="21"/>
+<wire x1="24.13" y1="28.194" x2="24.13" y2="1.524" width="0" layer="21"/>
+<wire x1="24.13" y1="1.524" x2="22.86" y2="0.254" width="0" layer="21" curve="-90"/>
+<wire x1="22.86" y1="0.254" x2="10.16" y2="0.254" width="0" layer="21"/>
+<wire x1="10.16" y1="0.254" x2="8.89" y2="1.524" width="0" layer="21" curve="-90"/>
+<wire x1="0" y1="0" x2="24.892" y2="0" width="0.2032" layer="20"/>
+<wire x1="24.892" y1="0" x2="24.892" y2="33.274" width="0.2032" layer="20"/>
+<wire x1="24.892" y1="33.274" x2="0" y2="33.274" width="0.2032" layer="20"/>
+<wire x1="0" y1="33.274" x2="0" y2="0" width="0.2032" layer="20"/>
 </plain>
 <attributes>
@@
 <pass name="Default">
 <param name="RoutingGrid" value="50mil"/>
-<param name="AutoGrid" value="1"/>
-<param name="Efforts" value="0"/>
-<param name="TopRouterVariant" value="1"/>
 <param name="tpViaShape" value="round"/>
-<param name="PrefDir.1" value="a"/>
+<param name="PrefDir.1" value="|"/>
 <param name="PrefDir.2" value="0"/>
 <param name="PrefDir.3" value="0"/>
@@
 <param name="PrefDir.14" value="0"/>
 <param name="PrefDir.15" value="0"/>
-<param name="PrefDir.16" value="a"/>
+<param name="PrefDir.16" value="-"/>
 <param name="cfVia" value="8"/>
 <param name="cfNonPref" value="5"/>
@@
 </autorouter>
 <elements>
-<element name="C1" library="SparkFun-Capacitors" package="CPOL-RADIAL-100UF-25V" value="4700" x="-26.67" y="5.08"/>
+<element name="C1" library="SparkFun-Capacitors" package="CPOL-RADIAL-100UF-25V" value="4700" x="5.08" y="9.906" rot="R180"/>
 <element name="FRAME1" library="SparkFun-Aesthetics" package="DUMMY" value="FRAME-LETTERNO_PACKAGE" x="-26.67" y="31.75">
 <attribute name="DESIGNER" value="Nobody" x="-26.67" y="31.75" size="1.778" layer="27" display="off"/>
 <attribute name="VERSION" value="v01" x="-26.67" y="31.75" size="1.778" layer="27" display="off"/>
 </element>
-<element name="JP1" library="SparkFun-Connectors" package="1X05" value="" x="-25.4" y="11.43"/>
-<element name="JP2" library="SparkFun-Connectors" package="1X05" value="" x="-25.4" y="16.51"/>
-<element name="PAD1" library="wirepad" package="1,6/0,8" value="WIREPAD1,6/0,8" x="-30.48" y="26.67"/>
-<element name="PAD2" library="wirepad" package="1,6/0,8" value="WIREPAD1,6/0,8" x="-17.78" y="31.75"/>
-<element name="PAD3" library="wirepad" package="1,6/0,8" value="WIREPAD1,6/0,8" x="-24.13" y="31.75"/>
-<element name="R1" library="SparkFun-Resistors" package="AXIAL-0.4" value="470" x="-19.05" y="21.59"/>
-<element name="R2" library="SparkFun-Resistors" package="AXIAL-0.4" value="330" x="-19.05" y="26.67"/>
-<element name="S1" library="SparkFun-Electromechanical" package="TACTILE-PTH" value="SWITCH-MOMENTARY-2PTH" x="-17.78" y="3.81">
-<attribute name="PROD_ID" value=" SWCH-08441" x="-17.78" y="3.81" size="1.778" layer="27" display="off"/>
+<element name="JP1" library="SparkFun-Connectors" package="1X05" value="" x="10.16" y="22.352" rot="R270"/>
+<element name="JP2" library="SparkFun-Connectors" package="1X05" value="" x="22.86" y="22.352" rot="R270"/>
+<element name="PAD1" library="wirepad" package="1,6/0,8" value="WIREPAD1,6/0,8" x="20.828" y="32.258"/>
+<element name="PAD2" library="wirepad" package="1,6/0,8" value="WIREPAD1,6/0,8" x="18.796" y="32.258"/>
+<element name="PAD3" library="wirepad" package="1,6/0,8" value="WIREPAD1,6/0,8" x="22.86" y="32.258"/>
+<element name="R1" library="SparkFun-Resistors" package="AXIAL-0.4" value="470" x="6.35" y="20.066" rot="R270"/>
+<element name="R2" library="SparkFun-Resistors" package="AXIAL-0.4" value="330" x="10.922" y="31.75"/>
+<element name="S1" library="SparkFun-Electromechanical" package="TACTILE-PTH" value="SWITCH-MOMENTARY-2PTH" x="4.572" y="3.302" rot="R180">
+<attribute name="PROD_ID" value=" SWCH-08441" x="4.572" y="3.302" size="1.778" layer="27" rot="R180" display="off"/>
 </element>
 </elements>
@@
 <contactref element="JP1" pad="1"/>
 <contactref element="R1" pad="P$1"/>
-<wire x1="-24.13" y1="21.59" x2="-25.4" y2="11.43" width="0" layer="19" extent="1-1"/>
+<wire x1="10.16" y1="22.352" x2="9.144" y2="22.352" width="0.254" layer="1"/>
+<wire x1="9.144" y1="22.352" x2="6.35" y2="25.146" width="0.254" layer="1"/>
 </signal>
 <signal name="N$2">
@@
 <contactref element="R1" pad="P$2"/>
 <contactref element="S1" pad="1"/>
-<wire x1="-22.86" y1="11.43" x2="-21.0312" y2="6.0706" width="0" layer="19" extent="1-1"/>
-<wire x1="-13.97" y1="21.59" x2="-22.86" y2="11.43" width="0" layer="19" extent="1-1"/>
+<wire x1="6.35" y1="14.986" x2="10.16" y2="19.812" width="0" layer="19" extent="1-1"/>
+<wire x1="7.8232" y1="1.0414" x2="6.35" y2="14.986" width="0" layer="19" extent="1-1"/>
 </signal>
 <signal name="GND">
@@
 <contactref element="PAD3" pad="1"/>
 <contactref element="C1" pad="2"/>
-<wire x1="-21.0312" y1="1.5494" x2="-27.94" y2="5.08" width="0" layer="19" extent="1-1"/>
-<wire x1="-17.78" y1="16.51" x2="-27.94" y2="5.08" width="0" layer="19" extent="1-1"/>
-<wire x1="-24.13" y1="31.75" x2="-17.78" y2="16.51" width="0" layer="19" extent="1-1"/>
+<polygon width="0.254" layer="1" isolate="0.3048">
+<vertex x="0" y="0"/>
+<vertex x="0" y="33.274"/>
+<vertex x="24.892" y="33.274"/>
+<vertex x="24.892" y="0"/>
+</polygon>
 </signal>
 <signal name="N$4">
 <contactref element="JP1" pad="4"/>
 <contactref element="R2" pad="P$1"/>
-<wire x1="-24.13" y1="26.67" x2="-17.78" y2="11.43" width="0" layer="19" extent="1-1"/>
+<wire x1="10.16" y1="14.732" x2="5.842" y2="31.75" width="0" layer="19" extent="1-1"/>
 </signal>
 <signal name="DIN">
 <contactref element="PAD2" pad="1"/>
 <contactref element="R2" pad="P$2"/>
-<wire x1="-13.97" y1="26.67" x2="-17.78" y2="31.75" width="0" layer="19" extent="1-1"/>
+<wire x1="16.002" y1="31.75" x2="18.288" y2="31.75" width="0.254" layer="1"/>
+<wire x1="18.288" y1="31.75" x2="18.796" y2="32.258" width="0.254" layer="1"/>
 </signal>
 <signal name="USB+">
@@
 <contactref element="C1" pad="1"/>
 <contactref element="JP1" pad="5"/>
-<wire x1="-15.24" y1="11.43" x2="-25.4" y2="5.08" width="0" layer="19" extent="1-1"/>
-<wire x1="-30.48" y1="26.67" x2="-15.24" y2="11.43" width="0" layer="19" extent="1-1"/>
+<wire x1="10.16" y1="12.192" x2="20.828" y2="32.258" width="0" layer="19" extent="1-1"/>
+<wire x1="3.81" y1="9.906" x2="10.16" y2="12.192" width="0" layer="19" extent="1-1"/>
+</signal>
+<signal name="N$1">
+<polygon width="0.254" layer="16" isolate="0.3048">
+<vertex x="0" y="0"/>
+<vertex x="0" y="33.274"/>
+<vertex x="24.892" y="33.274"/>
+<vertex x="24.892" y="0"/>
+</polygon>
 </signal>
 </signals>

Commit message: board finished
Routing:
- net USB+: track 0.00 -> 32.2 mm
- net N$2: track 0.00 -> 23.7 mm
- net N$4: track 0.00 -> 21.1 mm
Other:
- board size 24.9 x 33.3 mm -> 24.9 x 34.3 mm
- board text added: "4700"
- board text added: "5V"
- board text added: "DOUT"
- board text added: "GND"
- board text added: "Justin Lewsader"
- board text added: "NeoPixel Contoller"
- board text added: "Trinket Placement"
- board text added: "Ver. 1"
Changed lines of the file:
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@@
 <layer number="23" name="tOrigins" color="15" fill="1" visible="yes" active="yes"/>
 <layer number="24" name="bOrigins" color="15" fill="1" visible="yes" active="yes"/>
-<layer number="25" name="tNames" color="7" fill="1" visible="yes" active="yes"/>
-<layer number="26" name="bNames" color="7" fill="1" visible="yes" active="yes"/>
+<layer number="25" name="tNames" color="7" fill="1" visible="no" active="yes"/>
+<layer number="26" name="bNames" color="7" fill="1" visible="no" active="yes"/>
 <layer number="27" name="tValues" color="7" fill="1" visible="yes" active="yes"/>
 <layer number="28" name="bValues" color="7" fill="1" visible="yes" active="yes"/>
@@
 <wire x1="22.86" y1="0.254" x2="10.16" y2="0.254" width="0" layer="21"/>
 <wire x1="10.16" y1="0.254" x2="8.89" y2="1.524" width="0" layer="21" curve="-90"/>
-<wire x1="0" y1="0" x2="24.892" y2="0" width="0.2032" layer="20"/>
-<wire x1="24.892" y1="0" x2="24.892" y2="33.274" width="0.2032" layer="20"/>
-<wire x1="24.892" y1="33.274" x2="0" y2="33.274" width="0.2032" layer="20"/>
-<wire x1="0" y1="33.274" x2="0" y2="0" width="0.2032" layer="20"/>
+<wire x1="0" y1="-0.508" x2="24.892" y2="-0.508" width="0.2032" layer="20"/>
+<wire x1="24.892" y1="-0.508" x2="24.892" y2="33.782" width="0.2032" layer="20"/>
+<wire x1="24.892" y1="33.782" x2="0" y2="33.782" width="0.2032" layer="20"/>
+<wire x1="0" y1="33.782" x2="0" y2="-0.508" width="0.2032" layer="20"/>
+<text x="18.542" y="7.112" size="1.778" layer="21" rot="R90">Trinket
+Placement</text>
+<text x="20.066" y="29.972" size="0.762" layer="21">5V</text>
+<text x="21.844" y="29.972" size="0.762" layer="21">GND</text>
+<text x="16.764" y="29.972" size="0.762" layer="21">DOUT</text>
+<text x="4.064" y="7.366" size="0.762" layer="21">4700</text>
+<text x="2.032" y="18.288" size="1.27" layer="21" rot="R90">NeoPixel Contoller</text>
+<text x="4.064" y="26.67" size="1.27" layer="21" rot="R90">Ver. 1</text>
+<text x="3.81" y="18.288" size="0.762" layer="21" rot="R90">Justin Lewsader</text>
 </plain>
 <attributes>
@@
 </class>
 </classes>
-<designrules name="default">
-<description language="de">&lt;b&gt;EAGLE Design Rules&lt;/b&gt;
-&lt;p&gt;
-Die Standard-Design-Rules sind so gewählt, dass sie für
-die meisten Anwendungen passen. Sollte ihre Platine
-besondere Anforderungen haben, treffen Sie die erforderlichen
-Einstellungen hier und speichern die Design Rules unter
-einem neuen Namen ab.</description>
-<description language="en">&lt;b&gt;EAGLE Design Rules&lt;/b&gt;
-&lt;p&gt;
-The default Design Rules have been set to cover
-a wide range of applications. Your particular design
-may have different requirements, so please make the
-necessary adjustments and save your customized
-design rules under a new name.</description>
+<designrules name="SparkFun-2-layer-STANDARD">
+<description language="en">&lt;b&gt;SparkFun 2 Layer Design Rule Checks - STANDARD/TIGHT/FAB-LIMIT&lt;/b&gt;
+&lt;p&gt;
+These rules have been curated by SparkFuns DFM commitee. After doing much research, communicating with our multiple fab houses, and getting quotes of various designs, we have compiled three DRU files.
+&lt;p&gt;
+&lt;b&gt;STANDARD:&lt;/b&gt; This is more of a &quot;best case scenario&quot; set of limitations. If your design has the space, and/or you have the time to work within these parameters, please do. Larger trace width and clearance makes for easier visual inspection of the PCB while troubleshooting (useful in production and to the end user). It also allows for better ability to hack a trace (if you are crazy enough to scrape away the mask and solder to a trace). Another thing to keep in mind is that more metal is just more robust.
+&lt;p&gt;
+&lt;b&gt;TIGHT:&lt;/b&gt; This is where cost comes into play. We have found that most fab houses begin to add extra charges when you go smaller than these specs. In some cases, going to less than 15 mil trace can increase the cost by 10%. (This is why we have set the min drill on this DRU to 15 mil) Same story for traces thinner than 7 mil. To avoid those extra charges, then stay within the rules of this DRU.
+&lt;p&gt;
+&lt;b&gt;FAB-LIMIT:&lt;/b&gt; These set of rules are at the very limit of most fab houses capabilities. You will pay more for these specs, and it should be used on designs that have a darned good reason to need 4 mil vias and 4 mil traces.
+&lt;p&gt;
+**NOTE Clearance, Distance, Sizes, and Restring are all set to different limits in each of these three DRU files. Please compare the files within the CAM job editor window of eagle to see all the numbers.
+&lt;p&gt;
+***NOTE, Please set your Net Classes to default (0mil for all settings), so that it won't effect the DRC when you run it with these settings.</description>
 <param name="layerSetup" value="(1*16)"/>
 <param name="mtCopper" value="0.035mm 0.035mm 0.035mm 0.035mm 0.035mm 0.035mm 0.035mm 0.035mm 0.035mm 0.035mm 0.035mm 0.035mm 0.035mm 0.035mm 0.035mm 0.035mm"/>
 <param name="mtIsolate" value="1.5mm 0.15mm 0.2mm 0.15mm 0.2mm 0.15mm 0.2mm 0.15mm 0.2mm 0.15mm 0.2mm 0.15mm 0.2mm 0.15mm 0.2mm"/>
-<param name="mdWireWire" value="8mil"/>
+<param name="mdWireWire" value="10mil"/>
 <param name="mdWirePad" value="8mil"/>
-<param name="mdWireVia" value="8mil"/>
+<param name="mdWireVia" value="10mil"/>
 <param name="mdPadPad" value="8mil"/>
-<param name="mdPadVia" value="8mil"/>
-<param name="mdViaVia" value="8mil"/>
+<param name="mdPadVia" value="10mil"/>
+<param name="mdViaVia" value="10mil"/>
 <param name="mdSmdPad" value="8mil"/>
 <param name="mdSmdVia" value="8mil"/>
@@
 <param name="mdViaViaSameLayer" value="8mil"/>
 <param name="mnLayersViaInSmd" value="2"/>
-<param name="mdCopperDimension" value="40mil"/>
+<param name="mdCopperDimension" value="8mil"/>
 <param name="mdDrill" value="8mil"/>
 <param name="mdSmdStop" value="0mil"/>
 <param name="msWidth" value="10mil"/>
-<param name="msDrill" value="24mil"/>
+<param name="msDrill" value="20mil"/>
 <param name="msMicroVia" value="9.99mm"/>
 <param name="msBlindViaRatio" value="0.5"/>
@@
 <param name="rlMinPadBottom" value="10mil"/>
 <param name="rlMaxPadBottom" value="20mil"/>
-<param name="rlMinViaOuter" value="8mil"/>
+<param name="rlMinViaOuter" value="10mil"/>
 <param name="rlMaxViaOuter" value="20mil"/>
-<param name="rlMinViaInner" value="8mil"/>
+<param name="rlMinViaInner" value="10mil"/>
 <param name="rlMaxViaInner" value="20mil"/>
 <param name="rlMinMicroViaOuter" value="4mil"/>
@@
 <param name="mlMinCreamFrame" value="0mil"/>
 <param name="mlMaxCreamFrame" value="0mil"/>
-<param name="mlViaStopLimit" value="0mil"/>
+<param name="mlViaStopLimit" value="20mil"/>
 <param name="srRoundness" value="0"/>
 <param name="srMinRoundness" value="0mil"/>
@@
 <param name="dpGapFactor" value="2.5"/>
 <param name="checkGrid" value="0"/>
-<param name="checkAngle" value="0"/>
+<param name="checkAngle" value="1"/>
 <param name="checkFont" value="1"/>
 <param name="checkRestrict" value="1"/>
@@
 <contactref element="R1" pad="P$2"/>
 <contactref element="S1" pad="1"/>
-<wire x1="6.35" y1="14.986" x2="10.16" y2="19.812" width="0" layer="19" extent="1-1"/>
-<wire x1="7.8232" y1="1.0414" x2="6.35" y2="14.986" width="0" layer="19" extent="1-1"/>
+<wire x1="6.35" y1="14.986" x2="6.35" y2="16.002" width="0.4064" layer="1"/>
+<wire x1="6.35" y1="16.002" x2="10.16" y2="19.812" width="0.4064" layer="1"/>
+<wire x1="6.35" y1="14.986" x2="6.35" y2="12.954" width="0.4064" layer="16"/>
+<wire x1="6.35" y1="12.954" x2="11.176" y2="8.128" width="0.4064" layer="16"/>
+<wire x1="11.176" y1="8.128" x2="11.176" y2="4.3942" width="0.4064" layer="16"/>
+<wire x1="11.176" y1="4.3942" x2="7.8232" y2="1.0414" width="0.4064" layer="16"/>
 </signal>
 <signal name="GND">
@@
 <contactref element="JP1" pad="4"/>
 <contactref element="R2" pad="P$1"/>
-<wire x1="10.16" y1="14.732" x2="5.842" y2="31.75" width="0" layer="19" extent="1-1"/>
+<wire x1="5.842" y1="31.75" x2="5.842" y2="30.988" width="0.4064" layer="1"/>
+<wire x1="5.842" y1="30.988" x2="12.954" y2="23.876" width="0.4064" layer="1"/>
+<wire x1="12.954" y1="23.876" x2="12.954" y2="17.526" width="0.4064" layer="1"/>
+<wire x1="12.954" y1="17.526" x2="10.16" y2="14.732" width="0.4064" layer="1"/>
 </signal>
 <signal name="DIN">
@@
 <contactref element="C1" pad="1"/>
 <contactref element="JP1" pad="5"/>
-<wire x1="10.16" y1="12.192" x2="20.828" y2="32.258" width="0" layer="19" extent="1-1"/>
-<wire x1="3.81" y1="9.906" x2="10.16" y2="12.192" width="0" layer="19" extent="1-1"/>
+<wire x1="20.828" y1="32.258" x2="20.828" y2="25.146" width="0.4064" layer="1"/>
+<wire x1="20.828" y1="25.146" x2="14.224" y2="18.542" width="0.4064" layer="1"/>
+<wire x1="14.224" y1="18.542" x2="14.224" y2="16.256" width="0.4064" layer="1"/>
+<wire x1="14.224" y1="16.256" x2="10.16" y2="12.192" width="0.4064" layer="1"/>
+<wire x1="3.81" y1="9.906" x2="3.81" y2="10.668" width="0.4064" layer="1"/>
+<wire x1="3.81" y1="10.668" x2="5.334" y2="12.192" width="0.4064" layer="1"/>
+<wire x1="5.334" y1="12.192" x2="10.16" y2="12.192" width="0.4064" layer="1"/>
 </signal>
 <signal name="N$1">
@@
 </board>
 </drawing>
+<compatibility>
+<note version="6.3" minversion="6.2.2" severity="warning">
+Since Version 6.2.2 text objects can contain more than one line,
+which will not be processed correctly with this version.
+</note>
+</compatibility>
 </eagle>
